File: electronics/pcb/saufanlage/saufanlage.sch (KiCad schematic (older format))
At the start: 53 parts, among them J1 Conn_GND, J10 Conn_01x08_Male, J11 Conn_01x08_Male, J12 Conn_01x08_Male, J13 Conn_02x03_Odd_Even, J14 Conn_02x18_Odd_Even, J15 Conn_01x10_Male, J16 Conn_01x08_Male, J17 Conn_01x08_Male, J18 Conn_Finger, J19 Conn_Relais, J2 PJ-031D, J20 Conn_NFC, J21 Conn_Flow1, J22 Conn_Scale1, J23 Conn_01x15_Male, J24 Conn_01x15_Male, J25 Conn_Flow2, J26 Conn_Flow3, J27 Conn_Scale2, J28 Conn_Flow4, J29 Conn_01x15_Male, J3 Conn_3V3, J30 Conn_01x15_Male, J31 Conn_01x15_Male, J32 Conn_01x15_Male, J33 Conn_7SegmentI2C, J34 Conn_Scale2, J35 Conn_Scale2, J4 Conn_5V, J5 Conn_02x08_Odd_Even, J6 Conn_02x08_Odd_Even, J7 Conn_01x20_Male, J8 Raspberry_Pi_2_3, J9 Conn_01x20_Male

Commit message: Add temperature sensors
Parts:
- J34: value Conn_Scale2 -> Conn_Scale3
- J35: value Conn_Scale2 -> Conn_Scale4
- R1, R2, R3, R4, R5, R6: value ERJ-1RHD1003C -> ERJ-6RBD1003V; footprint saufanlage:ERJ-1RHD1003C -> saufanlage:ERJ-6RBD1003V; symbol 2020-02-06_21-37-09:ERJ-1RHD1003C -> 2020-02-06_21-37-09:ERJ-6RBD1003V
Connections:
- net M_5V: no longer TH4.1
- net M_A3: no longer TH4.2
Other:
- moved on the sheet: TH4
Changed lines of the file:
@@
 P 11250 12900
 F 0 "J34" H 11400 12200 50  0000 C CNN
-F 1 "Conn_Scale2" H 11200 13350 50  0000 C CNN
+F 1 "Conn_Scale3" H 11200 13350 50  0000 C CNN
 F 2 "Connector_PinHeader_2.54mm:PinHeader_1x10_P2.54mm_Vertical" H 11250 12900 50  0001 C CNN
 F 3 "~" H 11250 12900 50  0001 C CNN
@@
 P 12350 12900
 F 0 "J35" H 12500 12200 50  0000 C CNN
-F 1 "Conn_Scale2" H 12300 13350 50  0000 C CNN
+F 1 "Conn_Scale4" H 12300 13350 50  0000 C CNN
 F 2 "Connector_PinHeader_2.54mm:PinHeader_1x10_P2.54mm_Vertical" H 12350 12900 50  0001 C CNN
 F 3 "~" H 12350 12900 50  0001 C CNN
@@
 N1_5V
 $Comp
-L 2020-02-06_21-37-09:ERJ-1RHD1003C R1
+L 2020-02-06_21-37-09:ERJ-6RBD1003V R1
 U 1 1 5F3878CC
 P 10550 14350
 F 0 "R1" H 10800 14588 60  0000 C CNN
-F 1 "ERJ-1RHD1003C" H 10800 14482 60  0000 C CNN
-F 2 "saufanlage:ERJ-1RHD1003C" H 10800 14015 60  0001 C CNN
+F 1 "ERJ-6RBD1003V" H 10800 14482 60  0000 C CNN
+F 2 "saufanlage:ERJ-6RBD1003V" H 10800 14015 60  0001 C CNN
 F 3 "" H 10550 14350 60  0000 C CNN
 	1    10550 14350
@@
 Temp1
 $Comp
-L 2020-02-06_21-37-09:ERJ-1RHD1003C R2
+L 2020-02-06_21-37-09:ERJ-6RBD1003V R2
 U 1 1 5F9150F5
 P 10550 15450
 F 0 "R2" H 10800 15688 60  0000 C CNN
-F 1 "ERJ-1RHD1003C" H 10800 15582 60  0000 C CNN
-F 2 "saufanlage:ERJ-1RHD1003C" H 10800 15115 60  0001 C CNN
+F 1 "ERJ-6RBD1003V" H 10800 15582 60  0000 C CNN
+F 2 "saufanlage:ERJ-6RBD1003V" H 10800 15115 60  0001 C CNN
 F 3 "" H 10550 15450 60  0000 C CNN
 	1    10550 15450
@@
 Temp2
 $Comp
-L 2020-02-06_21-37-09:ERJ-1RHD1003C R4
+L 2020-02-06_21-37-09:ERJ-6RBD1003V R4
 U 1 1 5F9967A0
 P 12100 15450
 F 0 "R4" H 12350 15688 60  0000 C CNN
-F 1 "ERJ-1RHD1003C" H 12350 15582 60  0000 C CNN
-F 2 "saufanlage:ERJ-1RHD1003C" H 12350 15115 60  0001 C CNN
+F 1 "ERJ-6RBD1003V" H 12350 15582 60  0000 C CNN
+F 2 "saufanlage:ERJ-6RBD1003V" H 12350 15115 60  0001 C CNN
 F 3 "" H 12100 15450 60  0000 C CNN
 	1    12100 15450
@@
 L Device:Thermistor_NTC TH4
 U 1 1 5F9967B5
-P 13050 15450
-F 0 "TH4" V 12760 15450 50  0000 C CNN
-F 1 "Thermistor_NTC" V 12851 15450 50  0000 C CNN
-F 2 "Connector_PinHeader_2.54mm:PinHeader_1x02_P2.54mm_Vertical" H 13050 15500 50  0001 C CNN
-F 3 "~" H 13050 15500 50  0001 C CNN
-	1    13050 15450
+P 14600 15600
+F 0 "TH4" V 14310 15600 50  0000 C CNN
+F 1 "Thermistor_NTC" V 14401 15600 50  0000 C CNN
+F 2 "Connector_PinHeader_2.54mm:PinHeader_1x02_P2.54mm_Vertical" H 14600 15650 50  0001 C CNN
+F 3 "~" H 14600 15650 50  0001 C CNN
+	1    14600 15600
 	0    1    1    0
 $EndComp
@@
 Temp4
 $Comp
-L 2020-02-06_21-37-09:ERJ-1RHD1003C R3
+L 2020-02-06_21-37-09:ERJ-6RBD1003V R3
 U 1 1 5FA19023
 P 12100 14350
 F 0 "R3" H 12350 14588 60  0000 C CNN
-F 1 "ERJ-1RHD1003C" H 12350 14482 60  0000 C CNN
-F 2 "saufanlage:ERJ-1RHD1003C" H 12350 14015 60  0001 C CNN
+F 1 "ERJ-6RBD1003V" H 12350 14482 60  0000 C CNN
+F 2 "saufanlage:ERJ-6RBD1003V" H 12350 14015 60  0001 C CNN
 F 3 "" H 12100 14350 60  0000 C CNN
 	1    12100 14350
@@
 Temp3
 $Comp
-L 2020-02-06_21-37-09:ERJ-1RHD1003C R5
+L 2020-02-06_21-37-09:ERJ-6RBD1003V R5
 U 1 1 5FAA058F
 P 13650 14350
 F 0 "R5" H 13900 14588 60  0000 C CNN
-F 1 "ERJ-1RHD1003C" H 13900 14482 60  0000 C CNN
-F 2 "saufanlage:ERJ-1RHD1003C" H 13900 14015 60  0001 C CNN
+F 1 "ERJ-6RBD1003V" H 13900 14482 60  0000 C CNN
+F 2 "saufanlage:ERJ-6RBD1003V" H 13900 14015 60  0001 C CNN
 F 3 "" H 13650 14350 60  0000 C CNN
 	1    13650 14350
@@
 Temp5
 $Comp
-L 2020-02-06_21-37-09:ERJ-1RHD1003C R6
+L 2020-02-06_21-37-09:ERJ-6RBD1003V R6
 U 1 1 5FB247A2
 P 13650 15450
 F 0 "R6" H 13900 15688 60  0000 C CNN
-F 1 "ERJ-1RHD1003C" H 13900 15582 60  0000 C CNN
-F 2 "saufanlage:ERJ-1RHD1003C" H 13900 15115 60  0001 C CNN
+F 1 "ERJ-6RBD1003V" H 13900 15582 60  0000 C CNN
+F 2 "saufanlage:ERJ-6RBD1003V" H 13900 15115 60  0001 C CNN
 F 3 "" H 13650 15450 60  0000 C CNN
 	1    13650 15450
