File: electronics/pcb/saufanlage/saufanlage.sch (KiCad schematic (older format))
At the start: 53 parts, among them J1 Conn_GND, J10 Conn_01x08_Male, J11 Conn_01x08_Male, J12 Conn_01x08_Male, J13 Conn_02x03_Odd_Even, J14 Conn_02x18_Odd_Even, J15 Conn_01x10_Male, J16 Conn_01x08_Male, J17 Conn_01x08_Male, J18 Conn_Finger, J19 Conn_Relais, J2 PJ-031D, J20 Conn_NFC, J21 Conn_Flow1, J22 Conn_Scale1, J23 Conn_01x15_Male, J24 Conn_01x15_Male, J25 Conn_Flow2, J26 Conn_Flow3, J27 Conn_Scale2, J28 Conn_Flow4, J29 Conn_01x15_Male, J3 Conn_3V3, J30 Conn_01x15_Male, J31 Conn_01x15_Male, J32 Conn_01x15_Male, J33 Conn_7SegmentI2C, J34 Conn_Scale3, J35 Conn_Scale4, J4 Conn_5V, J5 Conn_02x08_Odd_Even, J6 Conn_02x08_Odd_Even, J7 Conn_01x20_Male, J8 Raspberry_Pi_2_3, J9 Conn_01x20_Male

Commit message: Add caps
Parts:
- added C1, C10, C11, C12, C13, C14, C15, C16, C17, C2, C3, C4, C5, C6, C7, C8, C9: 08054D226MAT2A, Capacitor_SMD:C_0805_2012Metric_Pad1.15x1.40mm_HandSolder, symbol Device:C
- R1, R2, R3, R4, R5, R6: footprint saufanlage:ERJ-6RBD1003V -> Resistor_SMD:R_0805_2012Metric_Pad1.15x1.40mm_HandSolder
- renumbered J33 to J10, J18 to J11, J10 to J12, J11 to J13, J12 to J14, J20 to J15, J21 to J16, J13 to J17, J14 to J18, J25 to J19, J15 to J20, J16 to J21, J17 to J22, J22 to J23, J26 to J24, J28 to J25, J27 to J26, J34 to J27, J19 to J28, J23 to J29, J24 to J30, J35 to J31, J29 to J32, J30 to J33, J31 to J34, J32 to J35
Connections:
- net GND: now also C1.1, C10.1, C11.1, C12.1, C13.1, C14.1, C15.1, C16.1, C17.1, C2.1, C3.1, C4.1, C5.1, C6.1, C7.1, C8.1, C9.1; no longer J24.1 (Pin_1)
- net M_3V3: now also C1.2, C10.2, C13.2, C3.2, C4.2, C5.2, C6.2, C7.2, C8.2, C9.2
- net M_5V: now also TH4.1, C11.2, C12.2, C14.2, C15.2, C16.2, C17.2, C2.2
- net M_A3: now also TH4.2
Other:
- moved on the sheet: J11, J16, J19, J24, J25, TH4
