File: electronics/pcb/saufanlage/saufanlage.kicad_pcb (KiCad board)
At the start: 2 copper layers, 320.3 x 186.4 mm, 39 parts, among them J1 Conn_GND, J10 Conn_01x08_Male, J11 Conn_01x08_Male, J12 Conn_01x08_Male, J13 Conn_02x03_Odd_Even, J14 Conn_02x18_Odd_Even, J15 Conn_01x10_Male, J16 Conn_01x08_Male, J17 Conn_01x08_Male, J18 Conn_Finger, J19 Conn_Relais, J2 PJ-031D, J20 Conn_NFC, J21 Conn_Flow1, J22 Conn_Scale1, J23 Conn_01x15_Male, J24 Conn_01x15_Male, J25 Conn_Flow2, J26 Conn_Flow3, J27 Conn_Scale2, J28 Conn_Flow4, J29 Conn_01x15_Male, J3 Conn_3V3, J30 Conn_01x15_Male, J31 Conn_01x15_Male, J32 Conn_01x15_Male, J33 Conn_7SegmentI2C, J4 Conn_5V, J5 Conn_02x08_Odd_Even, J6 Conn_02x08_Odd_Even, J7 Conn_01x20_Male, J8 Raspberry_Pi_2_3, J9 Conn_01x20_Male

Commit message: Add temperature sensors
Parts:
- added J34: Conn_Scale3, Connector_PinHeader_2.54mm:PinHeader_1x10_P2.54mm_Vertical, F.Cu at (175.0, 165.0)
- added J35: Conn_Scale4, Connector_PinHeader_2.54mm:PinHeader_1x10_P2.54mm_Vertical, F.Cu at (175.0, 180.0)
- added R1: ERJ-6RBD1003V, saufanlage:ERJ-6RBD1003V, F.Cu at (197.0, 150.0)
- added R2: ERJ-6RBD1003V, saufanlage:ERJ-6RBD1003V, F.Cu at (197.0, 160.0)
- added R3: ERJ-6RBD1003V, saufanlage:ERJ-6RBD1003V, F.Cu at (197.0, 170.0)
- added R4: ERJ-6RBD1003V, saufanlage:ERJ-6RBD1003V, F.Cu at (197.0, 180.0)
- added R5: ERJ-6RBD1003V, saufanlage:ERJ-6RBD1003V, F.Cu at (197.0, 190.0)
- added R6: ERJ-6RBD1003V, saufanlage:ERJ-6RBD1003V, F.Cu at (197.0, 200.0)
- added TH1: Thermistor_NTC, Connector_PinHeader_2.54mm:PinHeader_1x02_P2.54mm_Vertical, F.Cu at (205.0, 150.0)
- added TH2: Thermistor_NTC, Connector_PinHeader_2.54mm:PinHeader_1x02_P2.54mm_Vertical, F.Cu at (205.0, 160.0)
- added TH3: Thermistor_NTC, Connector_PinHeader_2.54mm:PinHeader_1x02_P2.54mm_Vertical, F.Cu at (205.0, 170.0)
- added TH4: Thermistor_NTC, Connector_PinHeader_2.54mm:PinHeader_1x02_P2.54mm_Vertical, F.Cu at (205.0, 180.0)
- added TH5: Thermistor_NTC, Connector_PinHeader_2.54mm:PinHeader_1x02_P2.54mm_Vertical, F.Cu at (205.0, 190.0)
- added TH6: Thermistor_NTC, Connector_PinHeader_2.54mm:PinHeader_1x02_P2.54mm_Vertical, F.Cu at (205.0, 200.0)
- moved J13 107.1 mm to (192.0, 45.5)
- moved J33 95.3 mm to (184.4, 200.0)
- moved J19 84.5 mm to (205.6, 127.2)
- moved J20 84.1 mm to (164.6, 210.0)
- moved J18 60.9 mm to (160.5, 200.0)
- moved J25 58.1 mm to (112.3, 210.0)
- moved J21 56.9 mm to (112.3, 200.0)
- moved J28 56.0 mm to (130.0, 210.0)
- moved J26 54.8 mm to (130.0, 200.0)
- moved J27 35.8 mm to (130.0, 180.0)
- moved J22 23.9 mm to (130.0, 165.0)
- moved J4 17.8 mm to (80.0, 147.5), turned to 180 degrees
- moved J1 14.0 mm to (45.0, 147.5), turned to 180 degrees
- moved J3 12.9 mm to (62.5, 147.5), turned to 180 degrees
Connections:
- net M_D2 renamed Sc4_DT4
- net M_D22 renamed Sc1_DT4
- net M_D23 renamed Sc1_SCK4
- net M_D24 renamed Sc1_DT3
- net M_D25 renamed Sc1_SCK3
- net M_D26 renamed Sc1_DT2
- net M_D27 renamed Sc1_SCK2
- net M_D28 renamed Sc1_DT1
- net M_D29 renamed Sc1_SCK1
- net M_D3 renamed Sc4_SCK4
- net M_D30 renamed Sc2_DT4
- net M_D31 renamed Sc2_SCK4
- net M_D32 renamed Sc2_DT3
- net M_D33 renamed Sc2_SCK3
- net M_D34 renamed Sc2_DT2
- net M_D35 renamed Sc2_SCK2
- net M_D36 renamed Sc2_DT1
- net M_D37 renamed Sc2_SCK1
- net M_D38 renamed Sc3_DT4
- net M_D39 renamed Sc3_SCK4
- net M_D4 renamed Sc4_DT3
- net M_D43 renamed Sc3_SCK2
- net M_D44 renamed Sc3_DT1
- net M_D45 renamed Sc3_SCK1
- net M_D49 renamed NFC_RST
- net M_D5 renamed Sc4_SCK3
- net M_D50 renamed NFC_MISO
- net M_D51 renamed NFC_MOSI
- net M_D52 renamed NFC_SCK
- net M_D53 renamed NFC_SDA
- net M_D6 renamed Sc4_DT2
- net M_D7 renamed Sc4_SCK2
- net M_D8 renamed Sc4_DT1
- net M_D9 renamed Sc4_SCK1
- J10 pad 8: Net-(J10-Pad8) -> (no net)
- J14 pad 13: M_D42 -> Sc3_DT2
- J14 pad 15: M_D40 -> Sc3_DT3
- J14 pad 16: M_D41 -> Sc3_SCK3
- J19 pad 2: Net-(J19-Pad2) -> Relais4
- J19 pad 3: M_D42 -> Relais3
- J19 pad 4: M_D41 -> Relais2
- J19 pad 5: M_D40 -> Relais1
- J19 pad 6: M_5V -> N1_5V
- J23 pad 1: N1_D12 -> Relais2
- J23 pad 2: N1_D11 -> Relais3
- J23 pad 3: N1_D10 -> Relais4
- J24 pad 15: N1_D13 -> Relais1
- XA1 pad D40: M_D40 -> Sc3_DT3
- XA1 pad D41: M_D41 -> Sc3_SCK3
- XA1 pad D42: M_D42 -> Sc3_DT2
- XA2 pad D10: N1_D10 -> Relais4
- XA2 pad D11: N1_D11 -> Relais3
- XA2 pad D12: N1_D12 -> Relais2
- XA2 pad D13: N1_D13 -> Relais1
Routing:
- net Sc4_SCK1: track 6.38 -> 243.1 mm
- net Sc4_DT1: track 6.38 -> 203.3 mm
- net Sc4_SCK2: track 6.37 -> 196.2 mm
- net Sc4_DT2: track 6.37 -> 190.2 mm
- net Sc4_SCK3: track 6.37 -> 182.8 mm
- net Sc4_DT3: track 6.37 -> 177.7 mm
- net Sc4_SCK4: track 6.37 -> 174.1 mm
- net Sc4_DT4: track 6.37 -> 163.9 mm
- net M_A5: track 6.34 -> 128.5 mm
- net M_A4: track 6.34 -> 121.0 mm
- net N1_5V: track 5.08 -> 117.4 mm
- net M_A3: track 6.34 -> 113.6 mm
- net M_A2: track 6.34 -> 106.6 mm
- net M_5V: track 171.8 -> 270.3 mm, vias 2 -> 1
- net M_A1: track 6.34 -> 98.7 mm
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Other:
- board text added: "7Segment"
- board text added: "SCK"
- board text added: "SPI"
- board text added: "Scales"
- board text added: "Temperature Sensors"
- board text removed: "SPI_5V"
- board text removed: "Scale 1"
- board text removed: "Scale 2"

Commit message: Clean up tracks
Routing:
- net Sc4_SCK1: track 243.1 -> 209.6 mm
- net RPI_GPIO20: track 62.2 -> 85.5 mm
- net RPI_GPIO19: track 62.6 -> 80.3 mm
- net RPI_GPIO24: track 136.6 -> 146.7 mm
- net Relais1: track 61.4 -> 71.0 mm
- net Sc3_DT1: track 56.7 -> 65.1 mm
- net Sc1_SCK4: track 53.5 -> 61.3 mm
- net Sc1_DT4: track 51.0 -> 58.5 mm
- net Sc3_SCK1: track 48.1 -> 55.2 mm
- net Relais2: track 40.6 -> 47.3 mm
- net Sc1_SCK3: track 52.6 -> 58.6 mm
- net Sc3_DT2: track 55.7 -> 60.7 mm
- net RPI_GPIO22: track 111.7 -> 116.7 mm
- net Sc3_SCK2: track 46.9 -> 50.5 mm
- net Sc1_DT3: track 50.0 -> 53.4 mm
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