File: electronics/pcb/saufanlage/saufanlage.kicad_pcb (KiCad board)
At the start: 2 copper layers, 320.3 x 186.4 mm, 53 parts, among them J1 Conn_GND, J10 Conn_01x08_Male, J11 Conn_01x08_Male, J12 Conn_01x08_Male, J13 Conn_02x03_Odd_Even, J14 Conn_02x18_Odd_Even, J15 Conn_01x10_Male, J16 Conn_01x08_Male, J17 Conn_01x08_Male, J18 Conn_Finger, J19 Conn_Relais, J2 PJ-031D, J20 Conn_NFC, J21 Conn_Flow1, J22 Conn_Scale1, J23 Conn_01x15_Male, J24 Conn_01x15_Male, J25 Conn_Flow2, J26 Conn_Flow3, J27 Conn_Scale2, J28 Conn_Flow4, J29 Conn_01x15_Male, J3 Conn_3V3, J30 Conn_01x15_Male, J31 Conn_01x15_Male, J32 Conn_01x15_Male, J33 Conn_7SegmentI2C, J34 Conn_Scale3, J35 Conn_Scale4, J4 Conn_5V, J5 Conn_02x08_Odd_Even, J6 Conn_02x08_Odd_Even, J7 Conn_01x20_Male, J8 Raspberry_Pi_2_3, J9 Conn_01x20_Male

Commit message: Add caps
Parts:
- added C1: 08054D226MAT2A, Capacitor_SMD:C_0805_2012Metric_Pad1.15x1.40mm_HandSolder, B.Cu at (152.9, 196.3)
- added C10: 08054D226MAT2A, Capacitor_SMD:C_0805_2012Metric_Pad1.15x1.40mm_HandSolder, B.Cu at (152.1, 168.8)
- added C11: 08054D226MAT2A, Capacitor_SMD:C_0805_2012Metric_Pad1.15x1.40mm_HandSolder, B.Cu at (207.5, 150.0)
- added C12: 08054D226MAT2A, Capacitor_SMD:C_0805_2012Metric_Pad1.15x1.40mm_HandSolder, B.Cu at (207.5, 160.0)
- added C13: 08054D226MAT2A, Capacitor_SMD:C_0805_2012Metric_Pad1.15x1.40mm_HandSolder, B.Cu at (152.1, 183.4)
- added C14: 08054D226MAT2A, Capacitor_SMD:C_0805_2012Metric_Pad1.15x1.40mm_HandSolder, B.Cu at (207.5, 170.0)
- added C15: 08054D226MAT2A, Capacitor_SMD:C_0805_2012Metric_Pad1.15x1.40mm_HandSolder, B.Cu at (207.5, 180.0)
- added C16: 08054D226MAT2A, Capacitor_SMD:C_0805_2012Metric_Pad1.15x1.40mm_HandSolder, B.Cu at (207.5, 190.0)
- added C17: 08054D226MAT2A, Capacitor_SMD:C_0805_2012Metric_Pad1.15x1.40mm_HandSolder, B.Cu at (207.5, 200.0)
- added C2: 08054D226MAT2A, Capacitor_SMD:C_0805_2012Metric_Pad1.15x1.40mm_HandSolder, B.Cu at (176.7, 204.1)
- added C3: 08054D226MAT2A, Capacitor_SMD:C_0805_2012Metric_Pad1.15x1.40mm_HandSolder, B.Cu at (149.4, 213.8)
- added C4: 08054D226MAT2A, Capacitor_SMD:C_0805_2012Metric_Pad1.15x1.40mm_HandSolder, B.Cu at (107.1, 203.7)
- added C5: 08054D226MAT2A, Capacitor_SMD:C_0805_2012Metric_Pad1.15x1.40mm_HandSolder, B.Cu at (107.1, 213.8)
- added C6: 08054D226MAT2A, Capacitor_SMD:C_0805_2012Metric_Pad1.15x1.40mm_HandSolder, B.Cu at (107.1, 168.8)
- added C7: 08054D226MAT2A, Capacitor_SMD:C_0805_2012Metric_Pad1.15x1.40mm_HandSolder, B.Cu at (124.8, 203.6)
- added C8: 08054D226MAT2A, Capacitor_SMD:C_0805_2012Metric_Pad1.15x1.40mm_HandSolder, B.Cu at (124.8, 213.8)
- added C9: 08054D226MAT2A, Capacitor_SMD:C_0805_2012Metric_Pad1.15x1.40mm_HandSolder, B.Cu at (107.2, 183.9)
- R1, R2, R3, R4, R5, R6: footprint saufanlage:ERJ-6RBD1003V -> Resistor_SMD:R_0805_2012Metric_Pad1.15x1.40mm_HandSolder; moved to B.Cu
- moved R1 1.52 mm to (195.5, 150.0)
- moved R2 1.52 mm to (195.5, 160.0)
- moved R3 1.52 mm to (195.5, 170.0)
- moved R4 1.52 mm to (195.5, 180.0)
- moved R5 1.52 mm to (195.5, 190.0)
- moved R6 1.52 mm to (195.5, 200.0)
- moved TH1 1.52 mm to (203.5, 150.0)
- moved TH2 1.52 mm to (203.5, 160.0)
- moved TH3 1.52 mm to (203.5, 170.0)
- moved TH4 1.52 mm to (203.5, 180.0)
- moved TH5 1.52 mm to (203.5, 190.0)
- moved TH6 1.52 mm to (203.5, 200.0)
- renumbered J33 to J10, J18 to J11, J10 to J12, J11 to J13, J12 to J14, J20 to J15, J21 to J16, J13 to J17, J14 to J18, J25 to J19, J15 to J20, J16 to J21, J17 to J22, J22 to J23, J26 to J24, J28 to J25, J27 to J26, J34 to J27, J19 to J28, J23 to J29, J24 to J30, J35 to J31, J29 to J32, J30 to J33, J31 to J34, J32 to J35
Routing:
- net M_3V3: track 300.7 -> 327.3 mm
- net M_5V: track 272.0 -> 297.4 mm, vias 1 -> 2
- net RPI_GPIO23: track 120.3 -> 142.5 mm, vias 0 -> 1
- net M_Flow2: track 162.3 -> 180.7 mm
- net RPI_GPIO25: track 143.9 -> 126.1 mm
- net M_A0: track 91.7 -> 107.5 mm
- net +8V: track 418.3 -> 432.8 mm
- net M_A4: track 121.0 -> 134.6 mm
- net GND: track 165.2 -> 175.9 mm
- net M_Flow3: track 191.7 -> 201.8 mm
- net M_Flow4: track 191.5 -> 200.8 mm
- net RPI_GPIO5: track 63.0 -> 70.8 mm
- net MEGA_RX1: track 115.3 -> 121.0 mm
- net Sc4_SCK4: track 174.1 -> 169.5 mm
- net RPI_GPIO12: track 58.7 -> 62.2 mm
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