File: electronics/pcb/saufanlage/saufanlage.kicad_pcb (KiCad board)
At the start: 2 copper layers, 303.8 x 186.4 mm, 38 parts, among them J1 Conn_01x08_Male, J10 Conn_01x08_Male, J11 Conn_01x08_Male, J12 Conn_01x08_Male, J13 Conn_02x03_Odd_Even, J14 Conn_02x18_Odd_Even, J15 Conn_01x10_Male, J16 Conn_01x08_Male, J17 Conn_01x08_Male, J18 Conn_01x04, J19 Conn_01x06_Female, J2 Screw_Terminal_01x02, J20 Conn_01x07_Male, J21 Conn_01x03_Male, J22 Conn_01x10_Male, J23 Conn_01x15_Male, J24 Conn_01x15_Male, J25 Conn_01x03_Male, J26 Conn_01x03_Male, J27 Conn_01x10_Male, J28 Conn_01x03_Male, J29 Conn_01x15_Male, J3 Conn_01x08_Male, J30 Conn_01x15_Male, J31 Conn_01x15_Male, J32 Conn_01x15_Male, J4 Conn_01x08_Male, J5 Conn_02x08_Odd_Even, J6 Conn_02x08_Odd_Even, J7 Conn_01x20_Male, J8 Raspberry_Pi_2_3, J9 Conn_01x20_Male

Commit message: More brainz updates
Parts:
- moved J2 38.2 mm to (61.5, 223.5)
- moved J9 36.9 mm to (101.1, 48.9)
- moved J7 35.5 mm to (94.0, 97.2)
- moved J31 34.7 mm to (300.5, 92.1)
- moved J1 34.7 mm to (42.9, 133.6)
- moved J24 34.7 mm to (224.3, 56.5)
- moved PS2 34.7 mm to (63.2, 167.1)
- moved J15 34.7 mm to (117.6, 47.7)
- moved J16 34.7 mm to (117.6, 74.6)
- moved J26 34.7 mm to (177.0, 172.0)
- moved J28 34.7 mm to (177.0, 179.6)
- moved J3 34.7 mm to (53.1, 138.7)
- moved J4 34.7 mm to (62.7, 143.3)
- moved J5 34.7 mm to (64.3, 118.9)
- moved J6 34.7 mm to (38.9, 118.9)
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Connections:
- J23 pad 13: N1_RST2 -> N1_RST1
- J24 pad 3: N1_RST1 -> N1_RST2
- J29 pad 13: N2_RST2 -> N2_RST1
- J30 pad 3: N2_RST1 -> N2_RST2
- J31 pad 13: N3_RST2 -> N3_RST1
- J32 pad 3: N3_RST1 -> N3_RST2
Routing:
- net +8V: track 6.33 -> 381.6 mm
- net SCL: track 6.38 -> 261.4 mm
- net SDA: track 6.38 -> 255.3 mm
- net +5V: track 0.00 -> 200.0 mm
- net +3V3: track 0.00 -> 195.5 mm
- net RPI_GPIO25: track 0.00 -> 141.8 mm
- net RPI_GPIO24: track 0.00 -> 136.6 mm
- net RPI_GPIO4: track 0.00 -> 136.3 mm, vias 0 -> 1
- net RPI_GPIO17: track 0.00 -> 131.2 mm
- net RPI_GPIO18: track 0.00 -> 120.4 mm
- net RPI_GPIO23: track 0.00 -> 115.9 mm
- net RPI_GPIO22: track 0.00 -> 111.7 mm, vias 0 -> 1
- net RPI_GPIO10: track 0.00 -> 87.6 mm
- net RPI_GPIO9: track 0.00 -> 85.1 mm
- net M_3V3: track 257.1 -> 334.4 mm
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- added copper zone on B.Cu, net GND
- added copper zone on F.Cu, net GND
Other:
- board size 303.8 x 186.4 mm -> 320.3 x 186.4 mm
- board text added: "+12V"
- board text added: "10"
- board text added: "11"
- board text added: "12"
- board text added: "13"
- board text added: "14"
- board text added: "15"
- board text added: "16"
- board text added: "17"
- board text added: "18"
- board text added: "19"
- board text added: "20"
- board text added: "21"
- board text added: "22"
- board text added: "23"
- board text added: "24"
- board text added: "25"
- board text added: "26"
- board text added: "27"
- board text added: "3.3V"
- board text added: "5V"
- board text added: "5V Buck Converter LM2596"
- board text added: "7"
- board text added: "8"
- board text added: "8V Buck Converter LM2596"
- board text added: "9"
- board text added: "A0"
- board text added: "A1"
- board text added: "A10"
- board text added: "A11"
- board text added: "A12"
- board text added: "A13"
- board text added: "A14"
- board text added: "A15"
- board text added: "A2"
- board text added: "A3"
- board text added: "A4"
- board text added: "A5"
- board text added: "A6"
- board text added: "A7"
- board text added: "A8"
- board text added: "A9"
- board text added: "AREF"
- board text added: "D0"
- board text added: "D1"
- board text added: "D10"
- board text added: "D11"
- board text added: "D12"
- board text added: "D13"
- board text added: "D2"
- board text added: "D22"
- board text added: "D23"
- board text added: "D24"
- board text added: "D25"
- board text added: "D26"
- board text added: "D27"
- board text added: "D28"
- board text added: "D29"
- board text added: "D3"
- board text added: "D30"
- board text added: "D31"
- board text added: "D32"
- board text added: "D33"
- board text added: "D34"
- board text added: "D35"
- board text added: "D36"
- board text added: "D37"
- board text added: "D38"
- board text added: "D39"
- board text added: "D4"
- board text added: "D46"
- board text added: "D47"
- board text added: "D48"
- board text added: "D49"
- board text added: "D5"
- board text added: "D50"
- board text added: "D51"
- board text added: "D52"
- board text added: "D53"
- board text added: "D6"
- board text added: "D7"
- board text added: "D8"
- board text added: "D9"
- board text added: "IDSC"
- board text added: "IDSD"
- board text added: "IORF"
- board text added: "MISO"
- board text added: "MOSI"
- board text added: "RST1"
- board text added: "RST2"
- board text added: "RX0"
- board text added: "RX1"
- board text added: "RX2"
- board text added: "RX3"
- board text added: "RX4"
- board text added: "Relais 1"
- board text added: "Relais 2"
- board text added: "Relais 3"
- board text added: "Relais 4"
- board text added: "Relais 5"
- board text added: "Relais 6"
- board text added: "SCL"
- board text added: "SDA"
- board text added: "SPI_5V"
- board text added: "Saufanlage – Brainz board"
- board text added: "TX0"
- board text added: "TX1"
- board text added: "TX2"
- board text added: "VIN"
- board text added: "VOUT (+5V)"
- board text added: "VOUT (+8V)"
- board text added: "v01"
- board text added: "–"

Commit message: Backup commit
Parts:
- added J33: Conn_7SegmentI2C, Connector_PinHeader_2.54mm:PinHeader_1x04_P2.54mm_Vertical, F.Cu at (104.6, 147.8)
- J1: value Conn_01x08_Male -> Conn_GND
- J18: value Conn_01x04 -> Conn_Finger
- J19: value Conn_01x06_Female -> Conn_Relais
- J2: value Screw_Terminal_01x02 -> PJ-031D; footprint Connector_Phoenix_MC:PhoenixContact_MCV_1,5_2-G-3.81_1x02_P3.81mm_Vertical -> PJ-031D:CUI_PJ-031D
- J20: value Conn_01x07_Male -> Conn_NFC
- J21: value Conn_01x03_Male -> Conn_Flow1
- J22: value Conn_01x10_Male -> Conn_Scale1
- J25: value Conn_01x03_Male -> Conn_Flow2
- J26: value Conn_01x03_Male -> Conn_Flow3
- J27: value Conn_01x10_Male -> Conn_Scale2
- J28: value Conn_01x03_Male -> Conn_Flow4
- J3: value Conn_01x08_Male -> Conn_3V3
- J4: value Conn_01x08_Male -> Conn_5V
- moved J2 55.0 mm to (25.9, 181.6), turned to 180 degrees
Connections:
- net M_D10 renamed M_Flow1
- net M_D11 renamed M_Flow2
- net M_D12 renamed M_Flow3
- net M_D13 renamed M_Flow4
- J14 pad 11: RELAIS6 -> M_D44
- J14 pad 12: RELAIS5 -> M_D45
- J14 pad 13: RELAIS4 -> M_D42
- J14 pad 14: RELAIS3 -> M_D43
- J14 pad 15: RELAIS2 -> M_D40
- J14 pad 16: RELAIS1 -> M_D41
- J19 pad 1: RELAIS6 -> GND
- J19 pad 2: RELAIS5 -> Net-(J19-Pad2)
- J19 pad 3: RELAIS4 -> M_D42
- J19 pad 4: RELAIS3 -> M_D41
- J19 pad 5: RELAIS2 -> M_D40
- J19 pad 6: RELAIS1 -> M_5V
- J2 pad 1: GND -> +12V
- J2 pad 2: +12V -> GND
- XA1 pad D40: RELAIS1 -> M_D40
- XA1 pad D41: RELAIS2 -> M_D41
- XA1 pad D42: RELAIS3 -> M_D42
- XA1 pad D43: RELAIS4 -> M_D43
- XA1 pad D44: RELAIS5 -> M_D44
- XA1 pad D45: RELAIS6 -> M_D45
Routing:
- net SCL: track 261.4 -> 375.6 mm
- net SDA: track 255.3 -> 360.4 mm
- net GND: track 96.0 -> 185.9 mm
- net RELAIS6: track 81.6 -> 0.00 mm, vias 4 -> 0
- net M_5V: track 96.7 -> 171.8 mm, vias 1 -> 2
- net RELAIS4: track 70.5 -> 0.00 mm, vias 1 -> 0
- net RELAIS2: track 67.5 -> 0.00 mm
- net RELAIS1: track 64.5 -> 0.00 mm
- net RELAIS3: track 63.4 -> 0.00 mm
- net M_D40: track 0.00 -> 63.4 mm
- net RELAIS5: track 62.4 -> 0.00 mm
- net M_D42: track 0.00 -> 62.4 mm
- net M_D41: track 0.00 -> 59.8 mm
- net M_D43: track 0.00 -> 35.3 mm
- net +12V: track 77.1 -> 45.4 mm
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Other:
- board text added: "LED Matrix 1"
- board text added: "LED Matrix 2"
- board text added: "v0.1"
- board text removed: "v01"

Commit message: Backup commit
Parts:
- removed the J13 at (107.7, 111.5)
- removed the J18 at (197.6, 151.6)
- removed the J22 at (146.6, 147.8)
- removed the J25 at (161.8, 179.6)
- added C1: 08054D226MAT2A, Capacitor_SMD:C_0805_2012Metric_Pad1.15x1.40mm_HandSolder, B.Cu at (152.9, 196.3)
- added C10: 08054D226MAT2A, Capacitor_SMD:C_0805_2012Metric_Pad1.15x1.40mm_HandSolder, B.Cu at (152.1, 168.8)
- added C11: 08054D226MAT2A, Capacitor_SMD:C_0805_2012Metric_Pad1.15x1.40mm_HandSolder, B.Cu at (207.5, 150.0)
- added C12: 08054D226MAT2A, Capacitor_SMD:C_0805_2012Metric_Pad1.15x1.40mm_HandSolder, B.Cu at (207.5, 160.0)
- added C13: 08054D226MAT2A, Capacitor_SMD:C_0805_2012Metric_Pad1.15x1.40mm_HandSolder, B.Cu at (152.1, 183.4)
- added C14: 08054D226MAT2A, Capacitor_SMD:C_0805_2012Metric_Pad1.15x1.40mm_HandSolder, B.Cu at (207.5, 170.0)
- added C15: 08054D226MAT2A, Capacitor_SMD:C_0805_2012Metric_Pad1.15x1.40mm_HandSolder, B.Cu at (207.5, 180.0)
- added C16: 08054D226MAT2A, Capacitor_SMD:C_0805_2012Metric_Pad1.15x1.40mm_HandSolder, B.Cu at (207.5, 190.0)
- added C17: 08054D226MAT2A, Capacitor_SMD:C_0805_2012Metric_Pad1.15x1.40mm_HandSolder, B.Cu at (207.5, 200.0)
- added C2: 08054D226MAT2A, Capacitor_SMD:C_0805_2012Metric_Pad1.15x1.40mm_HandSolder, B.Cu at (176.7, 204.1)
- added C3: 08054D226MAT2A, Capacitor_SMD:C_0805_2012Metric_Pad1.15x1.40mm_HandSolder, B.Cu at (149.4, 213.8)
- added C4: 08054D226MAT2A, Capacitor_SMD:C_0805_2012Metric_Pad1.15x1.40mm_HandSolder, B.Cu at (107.1, 203.7)
- added C5: 08054D226MAT2A, Capacitor_SMD:C_0805_2012Metric_Pad1.15x1.40mm_HandSolder, B.Cu at (107.1, 213.8)
- added C6: 08054D226MAT2A, Capacitor_SMD:C_0805_2012Metric_Pad1.15x1.40mm_HandSolder, B.Cu at (107.1, 168.8)
- added C7: 08054D226MAT2A, Capacitor_SMD:C_0805_2012Metric_Pad1.15x1.40mm_HandSolder, B.Cu at (124.8, 203.6)
- added C8: 08054D226MAT2A, Capacitor_SMD:C_0805_2012Metric_Pad1.15x1.40mm_HandSolder, B.Cu at (124.8, 213.8)
- added C9: 08054D226MAT2A, Capacitor_SMD:C_0805_2012Metric_Pad1.15x1.40mm_HandSolder, B.Cu at (107.2, 183.9)
- added J11: Conn_Finger, Connector_PinHeader_2.54mm:PinHeader_1x04_P2.54mm_Vertical, F.Cu at (160.5, 200.0)
- added J17: Conn_02x03_Odd_Even, Connector_PinHeader_2.54mm:PinHeader_2x03_P2.54mm_Vertical, F.Cu at (192.0, 45.5)
- added J19: Conn_Flow2, Connector_PinHeader_2.54mm:PinHeader_1x03_P2.54mm_Vertical, F.Cu at (112.3, 210.0)
- added J23: Conn_Scale1, Connector_PinHeader_2.54mm:PinHeader_1x10_P2.54mm_Vertical, F.Cu at (130.0, 165.0)
- added J26: Conn_Scale2, Connector_PinHeader_2.54mm:PinHeader_1x10_P2.54mm_Vertical, F.Cu at (130.0, 180.0)
- added J31: Conn_Scale4, Connector_PinHeader_2.54mm:PinHeader_1x10_P2.54mm_Vertical, F.Cu at (175.0, 180.0)
- added R1: ERJ-6RBD1003V, Resistor_SMD:R_0805_2012Metric_Pad1.15x1.40mm_HandSolder, B.Cu at (195.5, 150.0)
- added R2: ERJ-6RBD1003V, Resistor_SMD:R_0805_2012Metric_Pad1.15x1.40mm_HandSolder, B.Cu at (195.5, 160.0)
- added R3: ERJ-6RBD1003V, Resistor_SMD:R_0805_2012Metric_Pad1.15x1.40mm_HandSolder, B.Cu at (195.5, 170.0)
- added R4: ERJ-6RBD1003V, Resistor_SMD:R_0805_2012Metric_Pad1.15x1.40mm_HandSolder, B.Cu at (195.5, 180.0)
- added R5: ERJ-6RBD1003V, Resistor_SMD:R_0805_2012Metric_Pad1.15x1.40mm_HandSolder, B.Cu at (195.5, 190.0)
- added R6: ERJ-6RBD1003V, Resistor_SMD:R_0805_2012Metric_Pad1.15x1.40mm_HandSolder, B.Cu at (195.5, 200.0)
- added TH1: Thermistor_NTC, Connector_PinHeader_2.54mm:PinHeader_1x02_P2.54mm_Vertical, F.Cu at (203.5, 150.0)
- added TH2: Thermistor_NTC, Connector_PinHeader_2.54mm:PinHeader_1x02_P2.54mm_Vertical, F.Cu at (203.5, 160.0)
- added TH3: Thermistor_NTC, Connector_PinHeader_2.54mm:PinHeader_1x02_P2.54mm_Vertical, F.Cu at (203.5, 170.0)
- added TH4: Thermistor_NTC, Connector_PinHeader_2.54mm:PinHeader_1x02_P2.54mm_Vertical, F.Cu at (203.5, 180.0)
- added TH5: Thermistor_NTC, Connector_PinHeader_2.54mm:PinHeader_1x02_P2.54mm_Vertical, F.Cu at (203.5, 190.0)
- added TH6: Thermistor_NTC, Connector_PinHeader_2.54mm:PinHeader_1x02_P2.54mm_Vertical, F.Cu at (203.5, 200.0)
- J27: value Conn_Scale2 -> Conn_Scale3
- moved J10 95.3 mm to (184.4, 200.0)
- moved J28 84.5 mm to (205.6, 127.2)
- moved J15 84.1 mm to (164.6, 210.0)
- moved J16 56.9 mm to (112.3, 200.0)
- moved J25 56.0 mm to (130.0, 210.0)
- moved J24 54.8 mm to (130.0, 200.0)
- moved J27 20.3 mm to (175.0, 165.0)
- moved J4 17.8 mm to (80.0, 147.5), turned to 180 degrees
- moved J1 14.0 mm to (45.0, 147.5), turned to 180 degrees
- moved J3 12.9 mm to (62.5, 147.5), turned to 180 degrees
- renumbered J33 to J10, J10 to J12, J11 to J13, J12 to J14, J20 to J15, J21 to J16, J14 to J18, J15 to J20, J16 to J21, J17 to J22, J26 to J24, J28 to J25, J19 to J28, J23 to J29, J24 to J30, J29 to J32, J30 to J33, J31 to J34, J32 to J35
Connections:
- net M_D2 renamed Sc4_DT4
- net M_D22 renamed Sc1_DT4
- net M_D23 renamed Sc1_SCK4
- net M_D24 renamed Sc1_DT3
- net M_D25 renamed Sc1_SCK3
- net M_D26 renamed Sc1_DT2
- net M_D27 renamed Sc1_SCK2
- net M_D28 renamed Sc1_DT1
- net M_D29 renamed Sc1_SCK1
- net M_D3 renamed Sc4_SCK4
- net M_D4 renamed Sc4_DT3
- net M_D49 renamed NFC_RST
- net M_D5 renamed Sc4_SCK3
- net M_D50 renamed NFC_MISO
- net M_D51 renamed NFC_MOSI
- net M_D52 renamed NFC_SCK
- net M_D53 renamed NFC_SDA
- net M_D6 renamed Sc4_DT2
- net M_D7 renamed Sc4_SCK2
- net M_D8 renamed Sc4_DT1
- net M_D9 renamed Sc4_SCK1
- J12 pad 8: Net-(J10-Pad8) -> (no net)
- J18 pad 11: M_D44 -> Sc3_DT1
- J18 pad 12: M_D45 -> Sc3_SCK1
- J18 pad 13: M_D42 -> Sc3_DT2
- J18 pad 14: M_D43 -> Sc3_SCK2
- J18 pad 15: M_D40 -> Sc3_DT3
- J18 pad 16: M_D41 -> Sc3_SCK3
- J18 pad 17: M_D38 -> Sc3_DT4
- J18 pad 18: M_D39 -> Sc3_SCK4
- J18 pad 19: M_D36 -> Sc2_DT1
- J18 pad 20: M_D37 -> Sc2_SCK1
- J18 pad 21: M_D34 -> Sc2_DT2
- J18 pad 22: M_D35 -> Sc2_SCK2
- J18 pad 23: M_D32 -> Sc2_DT3
- J18 pad 24: M_D33 -> Sc2_SCK3
- J18 pad 25: M_D30 -> Sc2_DT4
- J18 pad 26: M_D31 -> Sc2_SCK4
- J27 pad 2: M_D37 -> Sc3_SCK1
- J27 pad 3: M_D36 -> Sc3_DT1
- J27 pad 4: M_D35 -> Sc3_SCK2
- J27 pad 5: M_D34 -> Sc3_DT2
- J27 pad 6: M_D33 -> Sc3_SCK3
- J27 pad 7: M_D32 -> Sc3_DT3
- J27 pad 8: M_D31 -> Sc3_SCK4
- J27 pad 9: M_D30 -> Sc3_DT4
- J28 pad 2: Net-(J19-Pad2) -> Relais4
- J28 pad 3: M_D42 -> Relais3
- J28 pad 4: M_D41 -> Relais2
- J28 pad 5: M_D40 -> Relais1
- J28 pad 6: M_5V -> N1_5V
- J29 pad 1: N1_D12 -> Relais2
- J29 pad 2: N1_D11 -> Relais3
- J29 pad 3: N1_D10 -> Relais4
- J30 pad 15: N1_D13 -> Relais1
- XA1 pad D30: M_D30 -> Sc2_DT4
- XA1 pad D31: M_D31 -> Sc2_SCK4
- XA1 pad D32: M_D32 -> Sc2_DT3
- XA1 pad D33: M_D33 -> Sc2_SCK3
- XA1 pad D34: M_D34 -> Sc2_DT2
- XA1 pad D35: M_D35 -> Sc2_SCK2
- XA1 pad D36: M_D36 -> Sc2_DT1
- XA1 pad D37: M_D37 -> Sc2_SCK1
- XA1 pad D38: M_D38 -> Sc3_DT4
- XA1 pad D39: M_D39 -> Sc3_SCK4
- XA1 pad D40: M_D40 -> Sc3_DT3
- XA1 pad D41: M_D41 -> Sc3_SCK3
- XA1 pad D42: M_D42 -> Sc3_DT2
- XA1 pad D43: M_D43 -> Sc3_SCK2
- XA1 pad D44: M_D44 -> Sc3_DT1
- XA1 pad D45: M_D45 -> Sc3_SCK1
- XA2 pad D10: N1_D10 -> Relais4
- XA2 pad D11: N1_D11 -> Relais3
- XA2 pad D12: N1_D12 -> Relais2
- XA2 pad D13: N1_D13 -> Relais1
Routing:
- net Sc4_SCK1: track 6.38 -> 208.5 mm
- net Sc4_DT1: track 6.38 -> 202.3 mm
- net Sc4_DT3: track 6.37 -> 195.5 mm
- net Sc4_SCK2: track 6.37 -> 195.1 mm
- net Sc4_DT2: track 6.37 -> 189.4 mm
- net Sc4_SCK3: track 6.37 -> 182.0 mm
- net Sc4_SCK4: track 6.37 -> 169.5 mm
- net Sc4_DT4: track 6.37 -> 163.3 mm
- net M_A4: track 6.34 -> 134.6 mm
- net M_5V: track 171.8 -> 297.3 mm
- net M_A5: track 6.34 -> 130.5 mm
- net N1_5V: track 5.08 -> 115.1 mm
- net M_A3: track 6.34 -> 113.2 mm
- net M_A0: track 6.34 -> 107.5 mm
- net M_A2: track 6.34 -> 105.5 mm
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Other:
- outline, holes or cut-outs redrawn
- board text added: "7Segment"
- board text added: "SCK"
- board text added: "SPI"
- board text added: "Scales"
- board text added: "Temperature Sensors"
- board text removed: "SPI_5V"
- board text removed: "Scale 1"
- board text removed: "Scale 2"
