File: electronics/pcb/load_cells_connector_board/load_cells_connector_board.kicad_pcb (KiCad board)
At the start: 2 copper layers, 95 x 158.5 mm, 9 parts, among them J1 Conn_01x10_Male, J2 Conn_01x04_Male, J3 Conn_01x04_Male, J4 Conn_01x04_Male, J5 Conn_01x04_Male, U1 XFW-HX711, U2 XFW-HX711, U3 XFW-HX711, U4 XFW-HX711

Commit message: Backup commit
Connections:
- U1 pad 5: Net-(U1-Pad5) -> (no net)
- U1 pad 6: Net-(U1-Pad6) -> (no net)
- U2 pad 5: Net-(U2-Pad5) -> (no net)
- U2 pad 6: Net-(U2-Pad6) -> (no net)
- U3 pad 5: Net-(U3-Pad5) -> (no net)
- U3 pad 6: Net-(U3-Pad6) -> (no net)
- U4 pad 5: Net-(U4-Pad5) -> (no net)
- U4 pad 6: Net-(U4-Pad6) -> (no net)
Routing:
- net VCC: track 235.2 -> 226.6 mm
- net Net-(J1-Pad9): track 49.8 -> 53.8 mm
Other:
- board text added: "1"
- board text added: "2"
- board text added: "3"
- board text added: "4"
- board text added: "A+"
- board text added: "A-"
- board text added: "DT"
- board text added: "E+"
- board text added: "E-"
- board text added: "GND"
- board text added: "SCK"
- board text added: "Vcc"
