File: electronics/pcb/load_cells_connector_board/load_cells_connector_board.sch (KiCad schematic (older format))
At the start: 9 parts, among them J1 Conn_01x10_Male, J2 Conn_01x04_Male, J3 Conn_01x04_Male, J4 Conn_01x04_Male, J5 Conn_01x04_Male, U1 XFW-HX711, U2 XFW-HX711, U3 XFW-HX711, U4 XFW-HX711

Commit message: Backup commit
Connections:
- no-connect marks 0 -> 8
Changed lines of the file:
@@
 Wire Wire Line
 	3050 3050 2700 3050
+NoConn ~ 4900 1650
+NoConn ~ 4900 1750
+NoConn ~ 4900 2600
+NoConn ~ 4900 2700
+NoConn ~ 4900 3700
+NoConn ~ 4900 3800
+NoConn ~ 4900 4800
+NoConn ~ 4900 4900
 $EndSCHEMATC
